File: Modified Files/V3/motherboard v3/motherboard v3.kicad_sch (KiCad schematic)
At the start: 60 parts, among them J1 Conn_01x02, J2 DuPont Connector, J2 JTAG_TC2030, SW1 Boot, U1 XC6206, U2 X05A26H12G, U3 RP2040, U4 W25Q128JVS, Y1 12MHz

Commit message: skipping v2 straight to v3
Parts:
- removed SW2, SW3, SW4, SW5, SW6, SW7, SW8: ~, Buttons:RanaTadpole, symbol ranatadpole:RanaTadpole
- added C17: 100nF, Capacitor_SMD:C_0402_1005Metric, symbol Device:C_Small
- added SW1: SW_Push, Connector_JST:JST_PH_S2B-PH-K_1x02_P2.00mm_Horizontal, symbol Switch:SW_Push
- added SW3, SW4: SW_Push, Button_Switch_THT:SW_PUSH_6mm_H5mm, symbol Switch:SW_Push
- renumbered SW20 to SW10, SW14 to SW11, SW18 to SW12, SW11 to SW13, SW21 to SW14, SW12 to SW16, SW16 to SW17, SW9 to SW5, SW19 to SW6, SW13 to SW7, SW17 to SW8, SW10 to SW9, U2 to U4
Connections:
- net LEFT is gone; now on net C_UP: U3.6 (GPIO4)
- net M1 is gone; now on net C_LT: U3.8 (GPIO6)
- net M2 is gone; now on net A: U3.9 (GPIO7)
- net +3V3: now also C17.1
- net A: no longer U3.17 (GPIO14)
- net B: now also U3.34 (GPIO22); no longer U3.38 (GPIO26/ADC0)
- net C_DN: now also U3.11 (GPIO8); no longer U3.18 (GPIO15)
- net C_LT: no longer U3.16 (GPIO13)
- net C_RT: now also U3.7 (GPIO5); no longer U3.27 (GPIO16)
- net C_UP: no longer U3.15 (GPIO12)
- net GND: now also SW1.2, C17.2, SW1.2, SW3.2, SW4.2; no longer SW1.1
- net L: now also U3.14 (GPIO11), SW1.1; no longer U3.7 (GPIO5)
- net LS: now also U3.28 (GPIO17); no longer U3.31 (GPIO20)
- net MS: now also U3.15 (GPIO12); no longer U3.29 (GPIO18)
- net R: now also U3.32 (GPIO21); no longer U3.39 (GPIO27/ADC1)
- net START: now also U3.38 (GPIO26/ADC0), SW3.1; no longer U3.2 (GPIO0)
- net X: now also U3.31 (GPIO20); no longer U3.32 (GPIO21)
- net Y: now also U3.30 (GPIO19); no longer U3.34 (GPIO22)
- net Z: now also U3.29 (GPIO18); no longer U3.30 (GPIO19)
- net ~{USB_BOOT}: now also SW1.1; no longer SW1.2
- net CS_SPI: now reaches U3.3 (GPIO1)
- net DOWN renamed Tx
- net RIGHT renamed CLK
- net UP renamed MOD
- net MOD: now also U3.27 (GPIO16); no longer U3.28 (GPIO17)
- new net D: SW4.1, U3.39 (GPIO27/ADC1)
- new net Rx: U3.2 (GPIO0)
- no-connect marks 26 -> 20
Other:
- added sheet Stickbox (stickbox.kicad_sch)
- moved on the sheet: C10, C11, C12, C13, C14, C15, C16, C17, C9, J2, R7, R8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
