File: Modified Files/V3/motherboard v3/motherboard v3.kicad_pcb (KiCad board)
At the start: 2 copper layers, 172 x 107 mm, 66 parts, among them J1 Conn_01x02, J2 JTAG_TC2030, J3 DuPont Connector, SW1 SW_Push, SW2 Boot, SW3 SW_Push, SW4 SW_Push, U1 RP2040, U2 W25Q128JVS, U3 XC6206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

Commit message: V3/4 cad
Parts:
- moved H1 98.2 mm to (141.0, 22.9)
- moved H3 98.2 mm to (140.5, 22.9)
- moved H4 81.1 mm to (73.6, 68.1)
- moved H2 81.1 mm to (73.2, 68.1)
- moved R9 19.4 mm to (93.0, 48.3), turned to 0 degrees
- moved C19 14.4 mm to (93.0, 52.1), turned to 180 degrees
- moved U5 12.3 mm to (71.1, 49.0)
- moved U7 7.68 mm to (80.2, 40.7)
- moved C13 7.47 mm to (99.8, 61.0), turned to 0 degrees
- moved C20 6.91 mm to (98.0, 52.1), turned to 180 degrees
- moved R10 6.29 mm to (98.0, 48.3), turned to 0 degrees
- moved U8 5.12 mm to (95.6, 58.4)
- moved SW1 2.02 mm to (88.6, 82.0)
- moved U4 1.22 mm to (110.2, 73.5)
- renumbered SW4 to SWe
Connections:
- C19 pad 1: Net-(U8-CH0) -> Net-(U8-CH1)
- C20 pad 1: Net-(U8-CH1) -> Net-(U8-CH0)
- R10 pad 2: Net-(U8-CH1) -> Net-(U8-CH0)
- R9 pad 2: Net-(U8-CH0) -> Net-(U8-CH1)
- U7 pad 3: unconnected-(U7-GND-Pad3) -> GND
Routing:
- net 3vDiode: track 180.6 -> 237.4 mm
- net CS_SPI: track 80.9 -> 118.4 mm, vias 1 -> 2
- net Tx: track 86.7 -> 121.1 mm, vias 1 -> 2
- net CLK: track 82.9 -> 114.7 mm, vias 1 -> 2
- net Rx: track 79.1 -> 110.2 mm, vias 1 -> 2
- net L: track 85.1 -> 113.5 mm
- net yHe: track 0.00 -> 21.9 mm
- net xHe: track 0.00 -> 21.8 mm
- net Net-(U8-CH0): track 0.00 -> 9.10 mm
- net Net-(U8-CH1): track 0.00 -> 8.08 mm
- net START: track 93.5 -> 95.1 mm
- net +5V: track 105.7 -> 106.7 mm
- net DATA: track 121.9 -> 122.9 mm
- net D: track 79.4 -> 80.1 mm
- net GND: track 54.7 -> 55.2 mm, vias 22 -> 23
Other:
- board size 172 x 107 mm -> 142.9 x 107 mm
