File: Modified Files/V3/motherboard v3/stickbox.kicad_sch (KiCad schematic)
At the start: 8 parts, among them U6 MCP3002, U7 DRV5055A2xDBZxQ1, U8 DRV5055A2xDBZxQ1, U9 Stickbox_Assembly_CStick

Commit message: V3/4 cad
Connections:
- net GND: now also U8.3 (GND)
- net at C18.1, R9.2: now also U6.3 (CH1); no longer U6.2 (CH0)
- net at C19.1, R10.2: now also U6.2 (CH0); no longer U6.3 (CH1)
Other:
- moved on the sheet: C18, C19, R10, R9, U6
